Commit message: Updated the model parameters

File: acrobot_description/models/acrobot.xacro (robot description, xacro)
@@ -9,9 +9,9 @@
     <link name="leg1">
         <inertial>
-            <mass value="436.312e-3"/>
-            <origin rpy="0 0 0" xyz="44.3396e-3 0 0"/>
-            <inertia ixx="3.60e-4" ixy="0.0" ixz="0.0"
-                     iyy="4.16e-3" iyz="0.0"
-                     izz="3.90e-3"/>
+            <mass value="460.566e-3"/>
+            <origin rpy="0 0 0" xyz="30.8842e-3 0.0259 0.3"/>
+            <inertia ixx="3.451e-4" ixy="0.0" ixz="0.0"
+                     iyy="2.565e-3" iyz="0.0"
+                     izz="2.308e-3"/>
         </inertial>
         <visual name="visual">
@@ -27,9 +27,9 @@
     <link name="leg2">
         <inertial>
-            <mass value="194.587e-3"/>
+            <mass value="226.876e-3"/>
             <origin rpy="0 0 0" xyz="-105.604e-3 0 0"/>
-            <inertia ixx="2.25e-4" ixy="0" ixz="0"
-                     iyy="2.53e-3" iyz="0"
-                     izz="2.33e-3"/>
+            <inertia ixx="2.816e-4" ixy="0" ixz="0"
+                     iyy="1.764e-3" iyz="0"
+                     izz="1.502e-3"/>
         </inertial>
         <visual name="visual">
@@ -46,5 +46,5 @@
         <parent link="base_link"/>
         <child link="leg1"/>
-        <origin rpy="0 ${PI/2} 0" xyz="0 0 0.354"/>
+        <origin rpy="0 ${PI/2} 0" xyz="0 0 0.390"/>
     </joint>
     <joint name="joint" type="revolute">

Commit message: Updated the pull request

File: acrobot_description/models/acrobot.xacro (robot description, xacro)
@@ -10,5 +10,5 @@
         <inertial>
             <mass value="460.566e-3"/>
-            <origin rpy="0 0 0" xyz="30.8842e-3 0.0259 0.3"/>
+            <origin rpy="0 0 0" xyz="30.8842e-3 0 0"/>
             <inertia ixx="3.451e-4" ixy="0.0" ixz="0.0"
                      iyy="2.565e-3" iyz="0.0"
@@ -46,5 +46,5 @@
         <parent link="base_link"/>
         <child link="leg1"/>
-        <origin rpy="0 ${PI/2} 0" xyz="0 0 0.390"/>
+        <origin rpy="0 ${PI/2} 0" xyz="0 0 0.360"/>
     </joint>
     <joint name="joint" type="revolute">
