Commit message: Updated model

File: acrobot_description/models/acrobot.urdf (robot description, URDF)
Before this commit: robot acrobot, 3 links, 2 joints
Links:
- added link leg1_extension, mass 48.358e-3; visual mesh filename=package://acrobot_description/meshes/leg_extension.stl scale=1 1 1
- link leg1: mass 256.815e-3 -> 436.312e-3
- link leg2: mass 166.44e-3 -> 194.587e-3
Joints:
- joint base_link: origin xyz=0 0 0.354 rpy=0 1.5707964 0 -> xyz=0 0 0.336 rpy=0 1.5707964 0
- joint joint: axis 0 1 0 -> (none); child leg2 -> leg1_extension; limit lower=-3.078760944 upper=3.078760944 effort=0.22 velocity=1.8 -> (none); origin xyz=0 0 0 rpy=0 0 0 -> xyz=0 0 167.5e-3 rpy=0 0 0; type revolute -> fixed

File: acrobot_description/models/acrobot.xacro (robot description, xacro)
@@ -5,12 +5,13 @@
     <xacro:property name="MOTOR_VELOCITY" value="1.8"/>
     <xacro:property name="PI" value="3.1415928"/>
+    <xacro:property name="MAXIMUM_ANGLE" value="${11*PI/12}"/>
     <link name="base_link" />
     <link name="leg1">
         <inertial>
-            <mass value="256.815e-3"/>
-            <origin rpy="0 0 0" xyz="89.16e-3 0 0"/>
-            <inertia ixx="6.16e-5" ixy="0.0" ixz="0.0"
-                     iyy="3.46e-3" iyz="0.0"
-                     izz="3.48e-3"/>
+            <mass value="436.312e-3"/>
+            <origin rpy="0 0 0" xyz="44.3396e-3 0 0"/>
+            <inertia ixx="3.60e-4" ixy="0.0" ixz="0.0"
+                     iyy="4.16e-3" iyz="0.0"
+                     izz="3.90e-3"/>
         </inertial>
         <visual name="visual">
@@ -26,9 +27,9 @@
     <link name="leg2">
         <inertial>
-            <mass value="166.44e-3"/>
-            <origin rpy="0 0 0" xyz="-183.44e-3 0 0"/>
-            <inertia ixx="1.94e-4" ixy="0" ixz="0"
-                     iyy="2.17e-3" iyz="0"
-                     izz="2.34e-3"/>
+            <mass value="194.587e-3"/>
+            <origin rpy="0 0 0" xyz="-105.604e-3 0 0"/>
+            <inertia ixx="2.25e-4" ixy="0" ixz="0"
+                     iyy="2.53e-3" iyz="0"
+                     izz="2.33e-3"/>
         </inertial>
         <visual name="visual">
@@ -53,5 +54,5 @@
         <axis xyz="0 1 0"/>
         <dynamics damping="${JOINT_DAMPING}" friction="${JOINT_FRICTION}" />
-        <limit effort="${MOTOR_TORQUE}" lower="-${PI*98/100}" upper="${PI*98/100}" velocity="${MOTOR_VELOCITY}"/>
+        <limit effort="${MOTOR_TORQUE}" lower="-${MAXIMUM_ANGLE}" upper="${MAXIMUM_ANGLE}" velocity="${MOTOR_VELOCITY}"/>
     </joint>
 </robot>

Commit message: More realistic steps for the motor

File: acrobot_description/models/acrobot.urdf (robot description, URDF)
Before this commit: robot acrobot, 4 links, 2 joints
Links:
- removed link leg1_extension
Joints:
- joint base_link: origin xyz=0 0 0.336 rpy=0 1.5707964 0 -> xyz=0 0 0.354 rpy=0 1.5707964 0
- joint joint: axis (none) -> 0 1 0; child leg1_extension -> leg2; limit (none) -> lower=-2.8797934 upper=2.8797934 effort=0.22 velocity=1.8; origin xyz=0 0 167.5e-3 rpy=0 0 0 -> xyz=0 0 0 rpy=0 0 0; type fixed -> revolute

Commit message: Done

File: acrobot_description/models/acrobot.urdf (robot description, URDF)
Before this commit: robot acrobot, 3 links, 2 joints
Links:
- link leg1: mass 436.312e-3 -> 460.566e-3
- link leg2: mass 194.587e-3 -> 226.876e-3
Joints:
- joint base_link: origin xyz=0 0 0.354 rpy=0 1.5707964 0 -> xyz=0 0 0.348 rpy=0 1.5707964 0

File: acrobot_description/models/acrobot.xacro (robot description, xacro)
@@ -10,8 +10,8 @@
         <inertial>
             <mass value="460.566e-3"/>
-            <origin rpy="0 0 0" xyz="30.8842e-3 0 0"/>
+            <origin rpy="0 0 0" xyz="30.4146e-3 0 0"/>
             <inertia ixx="3.451e-4" ixy="0.0" ixz="0.0"
-                     iyy="2.565e-3" iyz="0.0"
-                     izz="2.308e-3"/>
+                     iyy="2.45e-3" iyz="0.0"
+                     izz="2.19e-3"/>
         </inertial>
         <visual name="visual">
@@ -28,8 +28,8 @@
         <inertial>
             <mass value="226.876e-3"/>
-            <origin rpy="0 0 0" xyz="-105.604e-3 0 0"/>
-            <inertia ixx="2.816e-4" ixy="0" ixz="0"
-                     iyy="1.764e-3" iyz="0"
-                     izz="1.502e-3"/>
+            <origin rpy="0 0 0" xyz="-87.519e-3 0 0"/>
+            <inertia ixx="2.89e-4" ixy="0" ixz="0"
+                     iyy="1.66e-3" iyz="0"
+                     izz="1.41e-3"/>
         </inertial>
         <visual name="visual">
@@ -46,5 +46,5 @@
         <parent link="base_link"/>
         <child link="leg1"/>
-        <origin rpy="0 ${PI/2} 0" xyz="0 0 0.360"/>
+        <origin rpy="0 ${PI/2} 0" xyz="0 0 0.348"/>
     </joint>
     <joint name="joint" type="revolute">

Commit message: Better

File: acrobot_description/models/acrobot.urdf (robot description, URDF)
Before this commit: robot acrobot, 3 links, 2 joints
Links:
- link leg2: mass 226.876e-3 -> 109.617e-3

File: acrobot_description/models/acrobot.xacro (robot description, xacro)
@@ -27,9 +27,9 @@
     <link name="leg2">
         <inertial>
-            <mass value="226.876e-3"/>
-            <origin rpy="0 0 0" xyz="-87.519e-3 0 0"/>
-            <inertia ixx="2.89e-4" ixy="0" ixz="0"
-                     iyy="1.66e-3" iyz="0"
-                     izz="1.41e-3"/>
+            <mass value="109.617e-3"/>
+            <origin rpy="0 0 0" xyz="-92.3558e-3 0 0"/>
+            <inertia ixx="2.24e-4" ixy="0" ixz="0"
+                     iyy="1.60e-3" iyz="0"
+                     izz="1.38e-3"/>
         </inertial>
         <visual name="visual">
